File: weather_station_pico.kicad_sch (KiCad schematic)
At the start: 24 parts, among them J1 UART_DEBUG, J2 1984617, J3 STEMMA, J4 STEMMA_QT, J5 DS18B20, J6 1X7_HEADER, J7 RJ11, J8 RJ11, U1 PICO_W, U2 BME280

Commit message: Added footprints for antenna connector
Parts:
- added J7: 73412-0110, 734120110:MOLEX_73412-0110, symbol 73412-0110:73412-0110
- added U2: RFM69, RFM69:RFM69HCW_SPK, symbol 2024-03-24_21-06-40:COM-13909
- J1: value UART_DEBUG -> Conn_01x03
- U1: value PICO_W -> PICO
- renumbered H3 to H1, H4 to H2, H1 to H3, H2 to H4, J7 to J8, J8 to J9, U2 to U3
Connections:
- net GND: now also J1.3 (Pin_3), J7.2, U2.1 (GND), U2.10 (GND), U2.8 (GND); no longer J1.1 (Pin_1)
- net UART_TX: now also J1.1 (Pin_1); no longer J1.3 (Pin_3)
- net VCC: now also U2.13 (3.3V)
- net SPI0_MISO: now reaches U1.21 (GP16)
- net SPI0_MISO: now also U2.2 (MISO)
- net RFM69_CS: now reaches U1.22 (GP17)
- net RFM69_CS: now also U2.5 (NSS)
- net SPI0_CLK: now reaches U1.24 (GP18)
- net SPI0_CLK: now also U2.4 (SCK)
- net SPI0_MOSI: now reaches U1.25 (GP19)
- net SPI0_MOSI: now also U2.3 (MOSI)
- net RFM69_RESET: now reaches U1.26 (GP20)
- net RFM69_RESET: now also U2.6 (RESET)
- net FRM69_INTR: now reaches U1.27 (GP21)
- new net: J7.1, U2.9 (ANT)
- new net RFM69_INTR: U2.14 (DIO0)
- no-connect marks 31 -> 30
Other:
- note added: "RP PICO"
- note added: "UART"
- note removed: "RP PICO W"
- note removed: "UART DEBUG"
- moved on the sheet: H1, H2, H3, H4, U1
