File: station/rfm69.kicad_sch (KiCad schematic)
At the start: 3 parts, among them J3 73412-0110, U2 RFM69

Commit message: Added a reset button, status LEDs and broke out UART pins
Parts:
- renumbered J3 to J4
Changed lines of the file:
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@@
 		(dnp no)
 		(fields_autoplaced yes)
-		(property "Reference" "#PWR016"
+		(property "Reference" "#PWR020"
 			(at 194.31 90.17 0)
 			(effects
@@
 			(project "weather_station_pico"
 				(path "/8f1f45aa-e764-4c95-a223-c466cf9a95bf/f97a550c-f082-4b63-a8c6-81bc13221c5b"
-					(reference "#PWR016")
+					(reference "#PWR020")
 					(unit 1)
 				)
@@
 		(dnp no)
 		(fields_autoplaced yes)
-		(property "Reference" "#PWR017"
+		(property "Reference" "#PWR021"
 			(at 194.31 102.87 0)
 			(effects
@@
 			(project "weather_station_pico"
 				(path "/8f1f45aa-e764-4c95-a223-c466cf9a95bf/f97a550c-f082-4b63-a8c6-81bc13221c5b"
-					(reference "#PWR017")
+					(reference "#PWR021")
 					(unit 1)
 				)
@@
 		(dnp no)
 		(fields_autoplaced yes)
-		(property "Reference" "#PWR014"
+		(property "Reference" "#PWR018"
 			(at 170.18 90.17 0)
 			(effects
@@
 			(project "weather_station_pico"
 				(path "/8f1f45aa-e764-4c95-a223-c466cf9a95bf/f97a550c-f082-4b63-a8c6-81bc13221c5b"
-					(reference "#PWR014")
+					(reference "#PWR018")
 					(unit 1)
 				)
@@
 		(dnp no)
 		(fields_autoplaced yes)
-		(property "Reference" "J3"
+		(property "Reference" "J4"
 			(at 124.079 111.76 0)
 			(effects
@@
 			(project "weather_station_pico"
 				(path "/8f1f45aa-e764-4c95-a223-c466cf9a95bf/f97a550c-f082-4b63-a8c6-81bc13221c5b"
-					(reference "J3")
+					(reference "J4")
 					(unit 1)
 				)
@@
 		(dnp no)
 		(fields_autoplaced yes)
-		(property "Reference" "#PWR015"
+		(property "Reference" "#PWR019"
 			(at 170.18 127 0)
 			(effects
@@
 			(project "weather_station_pico"
 				(path "/8f1f45aa-e764-4c95-a223-c466cf9a95bf/f97a550c-f082-4b63-a8c6-81bc13221c5b"
-					(reference "#PWR015")
+					(reference "#PWR019")
 					(unit 1)
 				)
@@
 		(dnp no)
 		(fields_autoplaced yes)
-		(property "Reference" "#PWR013"
+		(property "Reference" "#PWR017"
 			(at 129.54 127 0)
 			(effects
@@
 			(project "weather_station_pico"
 				(path "/8f1f45aa-e764-4c95-a223-c466cf9a95bf/f97a550c-f082-4b63-a8c6-81bc13221c5b"
-					(reference "#PWR013")
-					(unit 1)
-				)
+					(reference "#PWR017")
+					(unit 1)
+				)
