File: station/weather_station_pico.kicad_pcb (KiCad board)
At the start: 2 copper layers, 70.5 x 76 mm, 36 parts, among them J1 UART, J10 Battery Charger, J2 I2C1_EXP, J3 I2C0_EXP, J4 73412-0110, J5 BME280, J6 WIND_SENSOR, J7 RAIN_SENSOR, J8 SOIL_MOISTURE, J9 SOIL_TEMP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

Commit message: V01 of the board complete
Parts:
- added G***: LOGO, WeatherStation:Logo, F.Cu at (147.4, 102.1)
- moved R5 3.95 mm to (149.4, 74.8)
- moved R6 3.95 mm to (145.5, 74.8)
- moved SW1 0.85 mm to (177.0, 103.0)
- turned D2 to 180 degrees
Connections:
- J4 pad 3: (no net) -> GND
Routing:
- net /I2C0_SDA: track 0.00 -> 98.3 mm, vias 0 -> 9
- net /I2C0_SCL: track 0.00 -> 91.3 mm, vias 0 -> 7
- net /I2C1_SCL: track 0.00 -> 88.0 mm, vias 0 -> 2
- net /I2C1_SDA: track 0.00 -> 81.7 mm, vias 0 -> 2
- net GND: track 65.4 -> 145.5 mm, vias 13 -> 71
- net /RFM69 Radio/RFM69_RESET: track 0.00 -> 45.9 mm, vias 0 -> 2
- net /ONE_WIRE: track 0.00 -> 43.9 mm
- net /UART0_RX: track 0.00 -> 41.6 mm, vias 0 -> 1
- net /RFM69 Radio/RFM69_INTR: track 0.00 -> 41.3 mm, vias 0 -> 2
- net /UART0_TX: track 0.00 -> 40.7 mm
- net /RFM69 Radio/RFM69_MOSI: track 0.00 -> 37.6 mm, vias 0 -> 2
- net /RFM69 Radio/RFM69_CLK: track 0.00 -> 29.8 mm, vias 0 -> 2
- net /STATUS_LED: track 0.00 -> 24.4 mm, vias 0 -> 1
- net /ERROR_LED: track 0.00 -> 22.0 mm, vias 0 -> 1
- net /RFM69 Radio/RFM69_CS: track 0.00 -> 21.9 mm, vias 0 -> 2
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Other:
- rule pad_to_mask_clearance: 0.0508 -> 0
- board text added: "+"
- board text added: "-"
- board text added: "10K"
- board text added: "1uF"
- board text added: "Error"
- board text added: "GND"
- board text added: "Light Sensor"
- board text added: "Pico Weather Station"
- board text added: "RX"
- board text added: "Reset"
- board text added: "Scott Perkins"
- board text added: "Status"
- board text added: "TX"
- board text added: "V01"

Commit message: Final Touches
Parts:
- moved R5 0.90 mm to (149.4, 75.7)
- moved R6 0.90 mm to (145.5, 75.7)
- moved C4 0.34 mm to (117.1, 72.7)
Routing:
- net +3.3V: track 264.0 -> 265.1 mm
- net Net-(D2-K): track 1.90 -> 2.80 mm
- net Net-(D1-K): track 1.90 -> 2.80 mm
- net /I2C0_SCL: track 91.3 -> 90.6 mm
Other:
- board text added: "220"
- board text added: "v01"
- board text removed: "V01"

Commit message: Fixed a defect where to wrong pins of the reset button were shorted together, causing the pico board to be in a constant reset state
Connections:
- SW1 pad 1: GND -> /RESET
- SW1 pad 4: /RESET -> GND
Routing:
- net GND: track 145.6 -> 151.1 mm, vias 71 -> 70
- net /RESET: track 25.6 -> 31.1 mm
Other:
- board text added: "v02"
- board text removed: "v01"
Changed lines of the file:
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@@
 			)
 		)
+		(property ki_fp_filters "1301.9314.24_SCH")
+		(sheetname "Root")
+		(sheetfile "weather_station_pico.kicad_sch")
 		(attr smd)
 		(fp_circle
@@
 			(size 2.1082 1.397)
 			(layers "F.Cu" "F.Paste" "F.Mask")
-			(net 1 "GND")
+			(net 50 "/RESET")
 			(pinfunction "1")
 			(pintype "unspecified")
@@
 			(size 2.1082 1.397)
 			(layers "F.Cu" "F.Paste" "F.Mask")
-			(net 50 "/RESET")
+			(net 1 "GND")
 			(pinfunction "4")
 			(pintype "unspecified")
@@
 		(sheetname "Root")
 		(sheetfile "weather_station_pico.kicad_sch")
-		(attr smd dnp)
+		(attr smd)
 		(fp_line
 			(start 0.227064 -0.735)
@@
 		(sheetname "Root")
 		(sheetfile "weather_station_pico.kicad_sch")
-		(attr smd dnp)
+		(attr smd)
 		(fp_line
 			(start 0.227064 -0.735)
@@
 		(sheetname "Root")
 		(sheetfile "weather_station_pico.kicad_sch")
-		(attr smd dnp)
+		(attr smd)
 		(fp_line
 			(start 0.227064 -0.735)
@@
 		(sheetname "Root")
 		(sheetfile "weather_station_pico.kicad_sch")
-		(attr smd dnp)
+		(attr smd)
 		(fp_line
 			(start 0.227064 -0.735)
@@
 		)
 	)
-	(gr_text "v01"
+	(gr_text "v02"
 		(at 122.845 137.8 0)
 		(layer "F.SilkS")
@@
 	)
 	(segment
+		(start 179.295001 97.95)
+		(end 179.295001 107.95)
+		(width 0.5)
+		(layer "F.Cu")
+		(net 1)
+	)
+	(segment
 		(start 118.2325 72.6)
 		(end 122.745 72.6)
@@
 	)
 	(segment
-		(start 174.794999 107.95)
-		(end 179.295001 107.95)
-		(width 1)
-		(layer "F.Cu")
-		(net 1)
-	)
-	(segment
 		(start 121.99 77.445)
 		(end 117.395 77.445)
@@
 	)
 	(via
-		(at 175.045 100.2)
-		(size 0.8)
-		(drill 0.4)
-		(layers "F.Cu" "B.Cu")
-		(free yes)
-		(net 1)
-	)
-	(via
 		(at 177.445 142.9)
 		(size 0.8)
@@
 	)
 	(segment
-		(start 174.744999 98)
+		(start 174.794999 107.95)
 		(end 174.794999 97.95)
 		(width 0.3)
@@
 	)
 	(segment
-		(start 174.794999 97.95)
-		(end 179.295001 97.95)
-		(width 1)
+		(start 174.744999 98)
+		(end 174.794999 97.95)
+		(width 0.3)
 		(layer "F.Cu")
 		(net 50)
